File: 4mosfets/4mosfets.kicad_pcb (KiCad board)
At the start: 2 copper layers, 36.8 x 17.1 mm, 22 parts, among them J1 Conn_01x04_Pin, J2 Conn_01x02_Pin, J3 Conn_01x02_Pin, J4 Conn_01x02_Pin, J5 Conn_01x02_Pin, J6 Conn_01x02_Pin, Q1 AO3400A, Q2 AO3400A, Q3 AO3400A, Q4 AO3400A

Commit message: updated pcb to have contacts closer to edge
Parts:
- moved J2 1.42 mm to (115.6, 75.6)
Routing:
- net /<NO NET>: track 53.7 -> 56.7 mm
- net Net-(D1-K): track 81.6 -> 83.4 mm
Changed lines of the file:
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@@
 	(footprint "Connector_PinHeader_2.54mm:PinHeader_1x02_P2.54mm_Vertical"
 		(layer "F.Cu")
-		(at 114.94 74.295 -90)
+		(at 115.575 75.565 -90)
 		(descr "Through hole straight pin header, 1x02, 2.54mm pitch, single row")
 		(tags "Through hole pin header THT 1x02 2.54mm single row")
@@
 	)
 	(segment
-		(start 119.555786 64.45)
-		(end 121.285 64.45)
+		(start 114.3 70.485)
+		(end 114.3 72.39)
 		(width 1)
 		(layer "B.Cu")
@@
 	)
 	(segment
-		(start 114.94 74.295)
-		(end 113.39 75.845)
+		(start 121.285 64.45)
+		(end 119.555786 64.45)
 		(width 1)
 		(layer "B.Cu")
@@
 	)
 	(segment
-		(start 113.665 73.367968)
-		(end 113.665 72.39)
+		(start 107.285 73.98)
+		(end 113.99 73.98)
 		(width 1)
 		(layer "B.Cu")
@@
 	)
 	(segment
-		(start 115.84 68.165786)
-		(end 119.555786 64.45)
+		(start 107.315 66.36)
+		(end 107.615 66.06)
 		(width 1)
 		(layer "B.Cu")
@@
 	)
 	(segment
-		(start 113.665 72.39)
-		(end 114.3 71.755)
+		(start 113.194214 66.06)
+		(end 114.3 67.165786)
 		(width 1)
 		(layer "B.Cu")
@@
 	)
 	(segment
-		(start 109.54 73.98)
-		(end 107.285 73.98)
+		(start 117.76 75.565)
+		(end 115.575 75.565)
 		(width 1)
 		(layer "B.Cu")
@@
 	)
 	(segment
-		(start 114.94 74.295)
-		(end 118.745 74.295)
+		(start 115.575 75.56)
+		(end 115.575 75.565)
 		(width 1)
 		(layer "B.Cu")
@@
 	)
 	(segment
-		(start 114.94 74.295)
-		(end 114.94 73.655)
+		(start 107.615 66.06)
+		(end 113.194214 66.06)
 		(width 1)
 		(layer "B.Cu")
@@
 	)
 	(segment
-		(start 114.94 74.295)
-		(end 114.592032 74.295)
+		(start 114.3 67.165786)
+		(end 114.3 70.485)
 		(width 1)
 		(layer "B.Cu")
@@
 	)
 	(segment
-		(start 114.94 73.655)
-		(end 115.84 72.755)
+		(start 119.555786 64.45)
+		(end 115.84 68.165786)
 		(width 1)
 		(layer "B.Cu")
@@
 	)
 	(segment
-		(start 107.615 66.06)
-		(end 107.315 66.36)
+		(start 113.99 73.98)
+		(end 115.575 75.565)
 		(width 1)
 		(layer "B.Cu")
@@
 	)
 	(segment
-		(start 118.745 74.295)
-		(end 120.97 72.07)
+		(start 114.3 72.39)
+		(end 115.575 73.665)
 		(width 1)
 		(layer "B.Cu")
@@
 	)
 	(segment
-		(start 114.3 71.755)
-		(end 114.3 67.165786)
+		(start 115.84 72.025)
+		(end 117.475 73.66)
 		(width 1)
 		(layer "B.Cu")
@@
 	)
 	(segment
-		(start 113.194214 66.06)
-		(end 107.615 66.06)
+		(start 115.575 73.665)
+		(end 115.575 75.565)
 		(width 1)
 		(layer "B.Cu")
@@
 	)
 	(segment
-		(start 111.405 75.845)
-		(end 109.54 73.98)
+		(start 117.475 73.66)
+		(end 115.575 75.56)
 		(width 1)
 		(layer "B.Cu")
@@
 	)
 	(segment
-		(start 120.97 72.07)
+		(start 117.76 75.565)
 		(end 121.255 72.07)
 		(width 1)
@@
 	)
 	(segment
-		(start 114.3 67.165786)
-		(end 113.194214 66.06)
-		(width 1)
-		(layer "B.Cu")
-		(net "/<NO NET>")
-	)
-	(segment
-		(start 115.84 72.755)
-		(end 115.84 68.165786)
+		(start 115.84 68.165786)
+		(end 115.84 72.025)
 		(width 1)
 		(layer "B.Cu")
@@
 	)
 	(segment
-		(start 114.592032 74.295)
-		(end 113.665 73.367968)
+		(start 125.0875 74.015)
+		(end 114.025 74.015)
 		(width 1)
-		(layer "B.Cu")
-		(net "/<NO NET>")
+		(layer "F.Cu")
+		(net "Net-(D1-K)")
 	)
 	(segment
-		(start 113.39 75.845)
-		(end 111.405 75.845)
+		(start 98.425 64.765)
+		(end 100.875 64.765)
 		(width 1)
-		(layer "B.Cu")
-		(net "/<NO NET>")
+		(layer "F.Cu")
+		(net "Net-(D1-K)")
 	)
 	(segment
-		(start 98.425 64.765)
-		(end 100.875 64.765)
+		(start 118.636262 72.745)
+		(end 113.31 72.745)
 		(width 1)
 		(layer "F.Cu")
@@
 	)
 	(segment
-		(start 121.976262 67.505)
-		(end 126.1975 67.505)
+		(start 102.235 63.405)
+		(end 106.585 63.405)
 		(width 1)
 		(layer "F.Cu")
@@
 	)
 	(segment
-		(start 111.197919 74.295)
-		(end 109.09 72.187081)
+		(start 109.09 65.91)
+		(end 109.09 72.26)
 		(width 1)
 		(layer "F.Cu")
@@
 	)
 	(segment
-		(start 112.4 74.295)
-		(end 112.4 73.092919)
+		(start 114.025 74.015)
+		(end 114.025 75.565)
 		(width 1)
 		(layer "F.Cu")
@@
 	)
 	(segment
-		(start 98.425 71.755)
-		(end 101.41 71.755)
+		(start 113.31 72.745)
+		(end 113.03 73.025)
 		(width 1)
 		(layer "F.Cu")
@@
 	)
 	(segment
-		(start 112.4 74.295)
-		(end 111.197919 74.295)
+		(start 113.035 73.03)
+		(end 113.035 75.565)
 		(width 1)
 		(layer "F.Cu")
@@
 	)
 	(segment
-		(start 112.4 74.295)
-		(end 111.13 75.565)
+		(start 110.813738 75.565)
+		(end 113.035 75.565)
 		(width 1)
 		(layer "F.Cu")
@@
 	)
 	(segment
-		(start 118.636262 72.745)
+		(start 119.8175 69.663762)
 		(end 119.8175 71.563762)
 		(width 1)
@@
 	)
 	(segment
-		(start 127.0225 74.3)
-		(end 126.1975 75.125)
+		(start 98.425 71.755)
+		(end 101.41 71.755)
 		(width 1)
 		(layer "F.Cu")
@@
 	)
 	(segment
-		(start 106.585 63.405)
-		(end 102.235 63.405)
+		(start 127.0225 74.3)
+		(end 126.1975 75.125)
 		(width 1)
 		(layer "F.Cu")
@@
 	)
 	(segment
-		(start 109.09 72.187081)
-		(end 109.09 65.91)
+		(start 119.8175 71.563762)
+		(end 118.636262 72.745)
 		(width 1)
 		(layer "F.Cu")
@@
 	)
 	(segment
-		(start 129.955 67.505)
-		(end 130.145 67.315)
+		(start 109.09 72.26)
+		(end 111.125 74.295)
 		(width 1)
 		(layer "F.Cu")
@@
 	)
 	(segment
-		(start 106.178738 70.93)
-		(end 102.235 70.93)
+		(start 126.1975 67.505)
+		(end 121.976262 67.505)
 		(width 1)
 		(layer "F.Cu")
@@
 	)
 	(segment
-		(start 111.13 75.565)
-		(end 110.49 75.565)
+		(start 129.955 67.505)
+		(end 130.145 67.315)
 		(width 1)
 		(layer "F.Cu")
@@
 	)
 	(segment
-		(start 110.49 75.241262)
-		(end 106.178738 70.93)
+		(start 114.025 75.565)
+		(end 113.035 75.565)
 		(width 1)
 		(layer "F.Cu")
@@
 	)
 	(segment
-		(start 112.747919 72.745)
-		(end 118.636262 72.745)
+		(start 126.1975 75.125)
+		(end 125.0875 74.015)
 		(width 1)
 		(layer "F.Cu")
@@
 	)
 	(segment
-		(start 109.09 65.91)
-		(end 106.585 63.405)
+		(start 106.178738 70.93)
+		(end 110.813738 75.565)
 		(width 1)
 		(layer "F.Cu")
@@
 	)
 	(segment
-		(start 126.1975 75.125)
-		(end 125.4775 75.845)
+		(start 111.125 74.295)
+		(end 111.765 74.295)
 		(width 1)
 		(layer "F.Cu")
@@
 	)
 	(segment
-		(start 112.4 74.295)
-		(end 112.4 74.855)
-		(width 1)
-		(layer "F.Cu")
-		(net "Net-(D1-K)")
-	)
-	(segment
-		(start 119.8175 71.563762)
-		(end 119.8175 69.663762)
+		(start 113.03 73.025)
+		(end 113.035 73.03)
 		(width 1)
 		(layer "F.Cu")
@@
 	)
 	(segment
-		(start 110.49 75.565)
-		(end 110.49 75.241262)
-		(width 1)
-		(layer "F.Cu")
-		(net "Net-(D1-K)")
-	)
-	(segment
-		(start 112.4 73.092919)
-		(end 112.747919 72.745)
-		(width 1)
-		(layer "F.Cu")
-		(net "Net-(D1-K)")
-	)
-	(segment
-		(start 112.4 74.295)
-		(end 112.355 74.25)
+		(start 101.41 71.755)
+		(end 102.235 70.93)
 		(width 1)
 		(layer "F.Cu")
@@
 	)
 	(segment
-		(start 125.4775 75.845)
-		(end 113.39 75.845)
+		(start 121.976262 67.505)
+		(end 119.8175 69.663762)
 		(width 1)
 		(layer "F.Cu")
@@
 	)
 	(segment
-		(start 112.4 74.855)
-		(end 113.39 75.845)
+		(start 111.765 74.295)
+		(end 113.035 75.565)
 		(width 1)
 		(layer "F.Cu")
@@
 	)
 	(segment
-		(start 119.8175 69.663762)
-		(end 121.976262 67.505)
+		(start 102.235 70.93)
+		(end 106.178738 70.93)
 		(width 1)
 		(layer "F.Cu")
@@
 	)
 	(segment
-		(start 101.41 71.755)
-		(end 102.235 70.93)
+		(start 106.585 63.405)
+		(end 109.09 65.91)
 		(width 1)
 		(layer "F.Cu")
